File: PowerComShield.sch (KiCad schematic (older format))
At the start: 36 parts, among them J1 Barrel_Jack, J3 Micro_SD_Card, J4 USB_B, K1 SANYOU_SRD_Form_C, P1 Digital, P10 CONN_01X01, P11 CONN_01X01, P12 CONN_01X01, P13 CONN_01X01, P2 Power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

Commit message: Add files via upload
Parts:
- removed Q3: Q_PMOS_GDS, TO254P1067X483X3124-3P:TO254P1067X483X3124-3P, symbol Device:Q_PMOS_GDS
- added D2: D_Zener, symbol Device:D_Zener
- added J10, J11, J8, J9: Conn_01x03, symbol Connector_Generic:Conn_01x03
- added J2, J7: Conn_01x02, symbol Connector_Generic:Conn_01x02
- added J5, J6: Conn_01x02, Connector_JST:JST_XH_B2B-XH-AM_1x02_P2.50mm_Vertical, symbol Connector_Generic:Conn_01x02
- added R2: 2.2kOhm, symbol Device:R
Connections:
- net +5V: now also Q4.3 (S), Q5.3 (S), Q6.3 (S), Q7.3 (S)
- net 10(**): now also J9.2 (Pin_2); no longer J3.2 (DAT3/CD)
- net 11(**): now also J8.2 (Pin_2)
- net 12(**): now also J3.2 (DAT3/CD); no longer U5.4 (DONE)
- net 13(**): now also D2.1 (K)
- net 2(**): now also Q4.1 (G)
- net 3(**): now also Q5.1 (G)
- net 4(**): now also Q6.1 (G)
- net 5(**): now also Q7.1 (G)
- net 6(**): now also J11.2 (Pin_2)
- net 9(**): now also J10.2 (Pin_2)
- net at C1.2, C2.2, J1.2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: now also J10.1 (Pin_1), J11.1 (Pin_1), J2.1 (Pin_1), J5.1 (Pin_1), J6.1 (Pin_1), J7.1 (Pin_1), J8.1 (Pin_1), J9.1 (Pin_1), R2.2
- net at U7.4 (AIN0): now also J8.3 (Pin_3)
- net at U7.5 (AIN1): now also J9.3 (Pin_3)
- net at U7.6 (AIN2): now also J10.3 (Pin_3)
- net at U7.7 (AIN3): now also J11.3 (Pin_3)
- net at Q4.2 (D): now also J7.2 (Pin_2)
- net at Q6.2 (D): now also J6.2 (Pin_2)
- net at Q7.2 (D): now also J2.2 (Pin_2)
- net at Q5.2 (D): now also J5.2 (Pin_2)
- new net: D2.2 (A), R2.1, U5.4 (DONE)
Other:
- moved on the sheet: D1, J4, Q4, Q5, Q6, Q7, U4, U6
